File: Programador_avr/FabISP/FabISP.sch (KiCad schematic (older format))
At the start: 14 parts, among them IC1 ATTINY44-SSU, M1 RESONATOR, M2 PINHD-1x02-SMD-HEADER, M3 MICRO-USB_1_64

Commit message: corrección de huellas y primeras rutas de pcb
Parts:
- C1: footprint fab:fab-C1206FAB -> Capacitor_SMD:C_1206_3216Metric
- JP1: footprint fab:fab-2X03SMD -> Connector_PinHeader_1.00mm:PinHeader_2x03_P1.00mm_Vertical_SMD
- M2: footprint fab:fab-1X02SMD -> Connector_PinHeader_1.00mm:PinHeader_2x01_P1.00mm_Vertical_SMD
- R1, R2, R3, R4, R5, R6: footprint fab:fab-R1206FAB -> Resistor_SMD:R_1206_3216Metric
Changed lines of the file:
@@
 F 0 "JP1" H 2350 1954 45  0000 C CNN
 F 1 "PINHD-2X3-SMD" H 2350 1870 45  0000 C CNN
-F 2 "fab:fab-2X03SMD" H 2330 1750 20  0001 C CNN
+F 2 "Connector_PinHeader_1.00mm:PinHeader_2x03_P1.00mm_Vertical_SMD" H 2330 1750 20  0001 C CNN
 F 3 "" H 2300 1600 50  0001 C CNN
 	1    2300 1600
@@
 F 0 "C1" V 1308 1678 45  0000 L CNN
 F 1 "1uF" V 1392 1678 45  0000 L CNN
-F 2 "fab:fab-C1206FAB" H 1330 1700 20  0001 C CNN
+F 2 "Capacitor_SMD:C_1206_3216Metric" H 1330 1700 20  0001 C CNN
 F 3 "" H 1300 1550 50  0001 C CNN
 	1    1300 1550
@@
 F 0 "R4" V 2758 3368 45  0000 L CNN
 F 1 "1K" H 2750 3200 45  0000 L CNN
-F 2 "fab:fab-R1206FAB" H 2830 3450 20  0001 C CNN
+F 2 "Resistor_SMD:R_1206_3216Metric" H 2830 3450 20  0001 C CNN
 F 3 "" H 2800 3300 50  0001 C CNN
 	1    2800 3300
@@
 F 0 "R5" V 3108 3668 45  0000 L CNN
 F 1 "499" V 3150 3400 45  0000 L CNN
-F 2 "fab:fab-R1206FAB" H 3180 3750 20  0001 C CNN
+F 2 "Resistor_SMD:R_1206_3216Metric" H 3180 3750 20  0001 C CNN
 F 3 "" H 3150 3600 50  0001 C CNN
 	1    3150 3600
@@
 F 0 "R3" V 6708 2318 45  0000 L CNN
 F 1 "100" H 6792 2318 45  0000 L CNN
-F 2 "fab:fab-R1206FAB" H 6780 2400 20  0001 C CNN
+F 2 "Resistor_SMD:R_1206_3216Metric" H 6780 2400 20  0001 C CNN
 F 3 "" H 6750 2250 50  0001 C CNN
 	1    6750 2250
@@
 F 0 "R6" V 6408 3818 45  0000 L CNN
 F 1 "100" H 6492 3818 45  0000 L CNN
-F 2 "fab:fab-R1206FAB" H 6480 3900 20  0001 C CNN
+F 2 "Resistor_SMD:R_1206_3216Metric" H 6480 3900 20  0001 C CNN
 F 3 "" H 6450 3750 50  0001 C CNN
 	1    6450 3750
@@
 F 0 "M2" H 2800 2200 45  0001 C CNN
 F 1 "PINHD-1x02-SMD-HEADER" H 2800 2200 45  0001 C CNN
-F 2 "fab:fab-1X02SMD" H 2830 2350 20  0001 C CNN
+F 2 "Connector_PinHeader_1.00mm:PinHeader_2x01_P1.00mm_Vertical_SMD" H 2830 2350 20  0001 C CNN
 F 3 "" H 2800 2200 50  0001 C CNN
 	1    2800 2200
@@
 F 0 "R2" V 6208 2318 45  0000 L CNN
 F 1 "10K" H 6292 2318 45  0000 L CNN
-F 2 "fab:fab-R1206FAB" H 6280 2400 20  0001 C CNN
+F 2 "Resistor_SMD:R_1206_3216Metric" H 6280 2400 20  0001 C CNN
 F 3 "" H 6250 2250 50  0001 C CNN
 	1    6250 2250
@@
 F 0 "R1" V 2958 1568 45  0000 L CNN
 F 1 "0" H 3042 1568 45  0000 L CNN
-F 2 "fab:fab-R1206FAB" H 3030 1650 20  0001 C CNN
+F 2 "Resistor_SMD:R_1206_3216Metric" H 3030 1650 20  0001 C CNN
 F 3 "" H 3000 1500 50  0001 C CNN
 	1    3000 1500

Commit message: correcciones sch y pcb
Other:
- note added: "Condensador\nde desacople"
- note added: "Conexión USB"
- note added: "Microcontrolador\ny conexiones"
- note added: "headers para conexiones externas"
- note added: "oscilador para el\nmicrocontrolador"
Changed lines of the file:
@@
 	-1   0    0    1
-$EndComp
-$Comp
-L fab:ATTINY44-SSU IC1
-U 1 1 5F8CD30F
-P 4100 3150
-F 0 "IC1" H 4950 4004 45  0000 C CNN
-F 1 "ATTINY44-SSU" H 4950 3920 45  0000 C CNN
-F 2 "fab:fab-SOIC-14_3.9x8.7mm_P1.27mm" H 4130 3300 20  0001 C CNN
-F 3 "" H 4100 3150 50  0001 C CNN
-	1    4100 3150
-	1    0    0    -1
 $EndComp
 Wire Wire Line
@@
 Wire Notes Line
 	3600 1150 6900 1150
+Text Notes 1400 4200 0    50   ~ 0
+Conexión USB
+Text Notes 1850 1150 0    50   ~ 0
+headers para conexiones externas
+$Comp
+L fab:ATTINY44-SSU IC1
+U 1 1 5F8CD30F
+P 4100 3150
+F 0 "IC1" H 4950 4004 45  0000 C CNN
+F 1 "ATTINY44-SSU" H 4950 3920 45  0000 C CNN
+F 2 "fab:fab-SOIC-14_3.9x8.7mm_P1.27mm" H 4130 3300 20  0001 C CNN
+F 3 "" H 4100 3150 50  0001 C CNN
+	1    4100 3150
+	1    0    0    -1
+$EndComp
+Text Notes 1100 2400 0    50   ~ 0
+Condensador\nde desacople
+Text Notes 3850 4100 0    50   ~ 0
+Microcontrolador\ny conexiones
+Text Notes 4250 1900 0    50   ~ 0
+oscilador para el\nmicrocontrolador
 $EndSCHEMATC

Commit message: correcciones
Parts:
- M1: value RESONATOR -> Reson.
Changed lines of the file:
@@
 P 5100 1500
 F 0 "M1" H 5100 1754 45  0000 C CNN
-F 1 "RESONATOR" H 5100 1670 45  0000 C CNN
+F 1 "Reson." H 5100 1670 45  0000 C CNN
 F 2 "fab:fab-EFOBM" H 5130 1650 20  0001 C CNN
 F 3 "" H 5100 1500 50  0001 C CNN

Commit message: Correcciones
Parts:
- removed R1: 0, Resistor_SMD:R_1206_3216Metric, symbol fab:RES-US1206FAB
- added M4: PINHD-1x02-SMD-HEADER, Connector_PinHeader_1.00mm:PinHeader_2x01_P1.00mm_Vertical_SMD, symbol fab:PINHD-1x02-SMD-HEADER
Connections:
- net D-: now also M4.2
- net at JP1.2: now also M4.1
Changed lines of the file:
@@
 Wire Wire Line
 	3150 3300 3150 3400
-Wire Wire Line
-	2500 1500 2800 1500
 $Comp
 L power:GND #PWR05
@@
 	1    6250 2250
 	0    1    1    0
-$EndComp
-$Comp
-L fab:RES-US1206FAB R1
-U 1 1 5F6E5992
-P 3000 1500
-F 0 "R1" V 2958 1568 45  0000 L CNN
-F 1 "0" H 3042 1568 45  0000 L CNN
-F 2 "Resistor_SMD:R_1206_3216Metric" H 3030 1650 20  0001 C CNN
-F 3 "" H 3000 1500 50  0001 C CNN
-	1    3000 1500
-	1    0    0    -1
 $EndComp
 NoConn ~ 6100 3650
@@
 Text Label 3350 1500 0    50   ~ 0
 D-
-Wire Wire Line
-	3200 1500 3350 1500
 $Comp
 L fab:MICRO-USB_1_64 M3
@@
 Text Notes 4250 1900 0    50   ~ 0
 oscilador para el\nmicrocontrolador
+$Comp
+L fab:PINHD-1x02-SMD-HEADER M4
+U 1 1 5FA881A7
+P 3450 1450
+F 0 "M4" H 3450 1450 45  0001 C CNN
+F 1 "PINHD-1x02-SMD-HEADER" H 3450 1450 45  0001 C CNN
+F 2 "Connector_PinHeader_1.00mm:PinHeader_2x01_P1.00mm_Vertical_SMD" H 3480 1600 20  0001 C CNN
+F 3 "" H 3450 1450 50  0001 C CNN
+	1    3450 1450
+	0    -1   -1   0
+$EndComp
+Wire Wire Line
+	2950 1500 2950 1450
+Wire Wire Line
+	2500 1500 2950 1500
+Wire Wire Line
+	3050 1450 3050 1500
+Wire Wire Line
+	3050 1500 3350 1500
 $EndSCHEMATC
